File: touch-controller.kicad_pcb (KiCad board)
At the start: 2 copper layers, 496.5 x 203.2 mm, 76 parts, among them J1 IR_DATA, J2 USB_C_Receptacle_USB2.0_16P, J3 IR_LED, J4 LED, K1 Conn_01x01, K10 Conn_01x01, K11 Conn_01x01, K12 Conn_01x01, K13 Conn_01x01, K14 Conn_01x01, K15 Conn_01x01, K16 Conn_01x01, K17 Conn_01x01, K18 Conn_01x01, K19 Conn_01x01, K2 Conn_01x01, K20 Conn_01x01, K21 Conn_01x01, K22 Conn_01x01, K23 Conn_01x01, K24 Conn_01x01, K25 Conn_01x01, K26 Conn_01x01, K27 Conn_01x01, K28 Conn_01x01, K29 Conn_01x01, K3 Conn_01x01, K30 Conn_01x01, K31 Conn_01x01, K32 Conn_01x01, K4 Conn_01x01, K5 Conn_01x01, K6 Conn_01x01, K7 Conn_01x01, K8 Conn_01x01, K9 Conn_01x01, Q1 BC818, Q2 BC818, SW1 FSM2JSMAATR, SW2 FSM2JSMAATR, U1 CH340C, U2 TVS0500DRVR, U3 TLV1117-33, U4 ESP32-S3-WROOM-1, U5 CAP1188-1-CP-TR, U6 CAP1188-1-CP-TR, U7 CAP1188-1-CP-TR, U8 CAP1188-1-CP-TR, U9 TPD2EUSB30DRTR

Commit message: Add ToF sensor & other changes (pcb broken)
Parts:
- removed the J1 at (52.1, 150.5)
- removed J3: IR_LED, Connector_PinHeader_2.54mm:PinHeader_1x03_P2.54mm_Horizontal
- added C10: 10uF, Capacitor_SMD:C_0805_2012Metric_Pad1.18x1.45mm_HandSolder, F.Cu at (371.2, 300.2)
- added C11: 0.1uF, Capacitor_SMD:C_0805_2012Metric_Pad1.18x1.45mm_HandSolder, F.Cu at (368.7, 300.2)
- added C3: 10uF, Capacitor_SMD:C_0805_2012Metric_Pad1.18x1.45mm_HandSolder, F.Cu at (215.5, 298.1)
- added C4: 0.1uF, Capacitor_SMD:C_0805_2012Metric_Pad1.18x1.45mm_HandSolder, F.Cu at (213.0, 298.1)
- added R10: 47k, Resistor_SMD:R_0805_2012Metric_Pad1.20x1.40mm_HandSolder, F.Cu at (286.0, 142.5)
- added R12: 47k, Resistor_SMD:R_0805_2012Metric_Pad1.20x1.40mm_HandSolder, F.Cu at (379.2, 296.7)
- added R6: 47k, Resistor_SMD:R_0805_2012Metric_Pad1.20x1.40mm_HandSolder, F.Cu at (223.5, 294.5)
- added R7: 47k, Resistor_SMD:R_0805_2012Metric_Pad1.20x1.40mm_HandSolder, F.Cu at (226.5, 299.5)
- added R8: 47k, Resistor_SMD:R_0805_2012Metric_Pad1.20x1.40mm_HandSolder, F.Cu at (286.0, 140.0)
- added U4: VL53L7CXV0GC/1, VL53L7CXV0GC-1:LGA16_OPTICAL-LINER_STM, F.Cu at (220.5, 298.1)
- added U7: VL53L7CXV0GC/1, VL53L7CXV0GC-1:LGA16_OPTICAL-LINER_STM, F.Cu at (376.2, 299.9)
- renumbered C9 to C12, C10 to C13, C3 to C2, C4 to C5, C5 to C6, C6 to C7, C7 to C8, C8 to C9, J2 to J1, J4 to J2, R6 to R11, R7 to R13, R8 to R14, R10 to R15, R11 to R16, R12 to R17, R13 to R18, R14 to R19, R15 to R20, R16 to R21, R17 to R22, U7 to U10, U8 to U11, U9 to U2, U2 to U3, U3 to U5, U4 to U6, U5 to U8, U6 to U9
Connections:
- U6 pad 20: IR_LED0 -> TOF_RESET
- U6 pad 21: IR_LED1 -> unconnected-(U6-GPIO13/TOUCH13/ADC2_CH2/FSPIQ/FSPIIO7/SUBSPIQ-Pad21)
- U6 pad 22: IR_LED2 -> unconnected-(U6-GPIO14/TOUCH14/ADC2_CH3/FSPIWP/FSPIDQS/SUBSPIWP-Pad22)
- U6 pad 38: IR_DATA1 -> unconnected-(U6-GPIO2/TOUCH2/ADC1_CH1-Pad38)
- U6 pad 39: IR_DATA0 -> unconnected-(U6-GPIO1/TOUCH1/ADC1_CH0-Pad39)
- U6 pad 4: IR_DATA2 -> unconnected-(U6-GPIO4/TOUCH4/ADC1_CH3-Pad4)
- U6 pad 5: IR_DATA3 -> unconnected-(U6-GPIO5/TOUCH5/ADC1_CH4-Pad5)
- U6 pad 6: IR_DATA4 -> TOF_LPN
- U6 pad 7: IR_DATA5 -> TOF_INT
Routing:
- net TOF_INT: track 0.00 -> 390.1 mm, vias 0 -> 5
- net TOF_LPN: track 0.00 -> 389.1 mm, vias 0 -> 2
- net +3.3V: track 542.6 -> 923.5 mm, vias 6 -> 9
- net GND: track 984.5 -> 1351.7 mm, vias 11 -> 12
- net TOF_RESET: track 0.00 -> 350.8 mm, vias 0 -> 5
- net SMDATA: track 455.5 -> 759.9 mm, vias 6 -> 9
- net SMCLK: track 409.4 -> 698.4 mm, vias 7 -> 10
- net IR_DATA0: track 262.1 -> 0.00 mm, vias 2 -> 0
- net IR_DATA1: track 261.3 -> 0.00 mm, vias 2 -> 0
- net IR_LED0: track 246.8 -> 0.00 mm
- net IR_LED1: track 244.5 -> 0.00 mm
- net IR_LED2: track 243.9 -> 0.00 mm
- net IR_DATA5: track 242.4 -> 0.00 mm
- net IR_DATA4: track 241.1 -> 0.00 mm
- net IR_DATA3: track 240.4 -> 0.00 mm
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Other:
- board size 496.5 x 203.2 mm -> 496.5 x 215.2 mm

Commit message: Partial pcb fix
Parts:
- removed the C1 at (273.6, 120.3)
- removed Q1, Q2: BC818, Package_TO_SOT_SMD:SOT-23
- removed the R1 at (262.8, 117.2)
- removed the R2 at (265.8, 117.2)
- removed the U1 at (273.5, 111.7)
- removed the U2 at (280.2, 105.5)
- added D1: LED, LED_SMD:LED_0805_2012Metric_Pad1.15x1.40mm_HandSolder, F.Cu at (287.5, 123.0)
- added R6: 62R, Resistor_SMD:R_0805_2012Metric_Pad1.20x1.40mm_HandSolder, F.Cu at (291.5, 123.0)
- added R7: 47k, Resistor_SMD:R_0805_2012Metric_Pad1.20x1.40mm_HandSolder, F.Cu at (279.5, 139.0)
- added U4: TPD1E05U06DYA, Diode_SMD:D_SOD-523, F.Cu at (278.3, 105.5)
- added U5: TPD1E05U06DYA, Diode_SMD:D_SOD-523, F.Cu at (284.7, 107.5)
- C8: renamed from C7; footprint Capacitor_THT:CP_Radial_D6.3mm_P2.50mm -> Capacitor_SMD:CP_Elec_6.3x5.8
- U3: value TVS0500DRVR -> TPD1E05U06DYA; footprint TVS0500DRVR:DRV0006A -> Diode_SMD:D_SOD-523
- moved U3 3.05 mm to (281.8, 105.5), turned to 0 degrees
- renumbered C3 to C1, C9 to C10, C12 to C11, C13 to C12, C10 to C2, C4 to C3, C11 to C4, C2 to C5, C5 to C6, C6 to C7, C8 to C9, D1 to D2, R6 to R1, R9 to R10, R10 to R11, R11 to R12, R12 to R2, R7 to R8, R8 to R9, U4 to U1, U7 to U2, U5 to U6, U6 to U7
Connections:
- R9 pad 1: TOF_LPN -> TOF_LPN1
- U1 pad A5: TOF_LPN -> TOF_LPN0
- U2 pad A5: TOF_LPN -> TOF_LPN1
- U3 pad 1: GND -> USB_D-
- U7 pad 13: unconnected-(U6-GPIO19/U1RTS/ADC2_CH8/CLK_OUT2/USB_D--Pad13) -> USB_D-
- U7 pad 14: unconnected-(U6-GPIO20/U1CTS/ADC2_CH9/CLK_OUT1/USB_D+-Pad14) -> USB_D+
- U7 pad 36: U0_RXD -> unconnected-(U7-U0RXD/GPIO44/CLK_OUT2-Pad36)
- U7 pad 37: UO_TXD -> unconnected-(U7-U0TXD/GPIO43/CLK_OUT1-Pad37)
- U7 pad 5: unconnected-(U6-GPIO5/TOUCH5/ADC1_CH4-Pad5) -> TOF_LPN0
- U7 pad 6: TOF_LPN -> TOF_LPN1
Routing:
- net TOF_LPN: track 389.1 -> 0.00 mm, vias 2 -> 0
- net TOF_LPN1: track 0.00 -> 281.1 mm, vias 0 -> 2
- net TOF_LPN0: track 0.00 -> 231.0 mm, vias 0 -> 2
- net GPIO0: track 77.9 -> 12.7 mm, vias 2 -> 0
- net U0_RXD: track 59.5 -> 0.00 mm, vias 2 -> 0
- net UO_TXD: track 56.0 -> 0.00 mm, vias 2 -> 0
- net +3.3V: track 923.5 -> 903.1 mm, vias 9 -> 10
- net EN: track 67.7 -> 49.0 mm
- net GND: track 1351.7 -> 1369.1 mm
- net DTR: track 16.8 -> 0.00 mm
- net RTS: track 13.3 -> 0.00 mm
- net Net-(Q1-B): track 9.71 -> 0.00 mm
- net USB_D-: track 18.6 -> 13.0 mm
- net Net-(Q2-B): track 5.18 -> 0.00 mm
- net Net-(D1-K): track 0.00 -> 4.02 mm
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